File: AS5040/AskelmoottoriV3.brd (EAGLE design)
At the start: 50.1 x 48.6 mm, 14 parts, among them IC1 AS5040

Commit message: Demo code
Parts:
- added C4: (no value), rcl:E1,8-4
Connections:
- new net N$15: C4.+, IC1.15
- net GND: now also C4.-
Routing:
- net N$15: track 0.00 -> 12.2 mm, vias 0 -> 1
- net GND: track 154.5 -> 158.4 mm
Changed lines of the file:
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@@
 <attribute name="VALUE" x="10.16" y="19.3294" size="1.27" layer="27" ratio="10" rot="R90"/>
+</element>
+<element name="C4" library="rcl" library_urn="urn:adsk.eagle:library:334" package="E1,8-4" package3d_urn="urn:adsk.eagle:package:23336/2" value="" x="21.59" y="32.0675" smashed="yes" rot="R90">
+<attribute name="NAME" x="20.828" y="34.2265" size="1.27" layer="25" ratio="10" rot="R90"/>
+<attribute name="SPICEPREFIX" value="C" x="21.59" y="32.0675" size="1.778" layer="27" rot="R90" display="off"/>
+<attribute name="VALUE" x="23.368" y="34.2265" size="1.27" layer="27" ratio="10" rot="R90"/>
 </element>
 </elements>
@@
 <wire x1="34.29" y1="39.37" x2="27.94" y2="39.37" width="0.1524" layer="16"/>
 <wire x1="25.695" y1="30.465" x2="25.695" y2="32.725" width="0.1524" layer="16"/>
-<wire x1="25.695" y1="32.725" x2="24.13" y2="34.29" width="0.1524" layer="16"/>
+<wire x1="25.4635" y1="32.9565" x2="24.13" y2="34.29" width="0.1524" layer="16"/>
 <wire x1="24.13" y1="34.29" x2="24.13" y2="35.56" width="0.1524" layer="16"/>
 <wire x1="25.695" y1="30.465" x2="25.695" y2="27.9175" width="0.1524" layer="16"/>
@@
 <via x="23.495" y="20.955" extent="1-16" drill="0.35"/>
 <via x="26.67" y="17.78" extent="1-16" drill="0.35"/>
+<contactref element="C4" pad="-"/>
+<wire x1="21.59" y1="32.9565" x2="25.4635" y2="32.9565" width="0.1524" layer="16"/>
+<wire x1="25.4635" y1="32.9565" x2="25.695" y2="32.725" width="0.1524" layer="16"/>
 </signal>
 <signal name="+5V">
@@
 <contactref element="U$1" pad="EN"/>
 <wire x1="34.29" y1="35.56" x2="28.28645" y2="35.56" width="0.1524" layer="1"/>
-<wire x1="28.28645" y1="35.56" x2="27.14345" y2="34.417" width="0.1524" layer="1"/>
-<wire x1="27.14345" y1="34.417" x2="22.987" y2="34.417" width="0.1524" layer="1"/>
-<wire x1="19.05" y1="30.48" x2="17.78" y2="30.48" width="0.1524" layer="1"/>
-<wire x1="22.987" y1="34.417" x2="19.05" y2="30.48" width="0.1524" layer="1"/>
+<wire x1="27.14345" y1="34.417" x2="28.28645" y2="35.56" width="0.1524" layer="1"/>
+<wire x1="17.78" y1="30.48" x2="20.4978" y2="33.1978" width="0.1524" layer="1"/>
+<wire x1="20.4978" y1="33.1978" x2="20.4978" y2="33.40890625" width="0.1524" layer="1"/>
+<wire x1="20.4978" y1="33.40890625" x2="21.50589375" y2="34.417" width="0.1524" layer="1"/>
+<wire x1="21.50589375" y1="34.417" x2="27.14345" y2="34.417" width="0.1524" layer="1"/>
 </signal>
 <signal name="N$11">
@@
 <wire x1="9.525" y1="12.7" x2="9.525" y2="16.51" width="0.1524" layer="1"/>
 </signal>
+<signal name="N$15">
+<contactref element="IC1" pad="15"/>
+<contactref element="C4" pad="+"/>
+<wire x1="21.59" y1="31.1785" x2="26.0985" y2="26.67" width="0.1524" layer="1"/>
+<wire x1="26.0985" y1="26.67" x2="27.94" y2="26.67" width="0.1524" layer="1"/>
+<via x="27.94" y="26.67" extent="1-16" drill="0.35"/>
+<wire x1="27.94" y1="26.67" x2="28.295" y2="27.025" width="0.1524" layer="16"/>
+<wire x1="28.295" y1="27.025" x2="28.295" y2="30.465" width="0.1524" layer="16"/>
+</signal>
 </signals>

Commit message: Update eagle files
Parts:
- removed C4: (no value), rcl:E1,8-4
- added C5: (no value), rcl:E2,5-5
Connections:
- new net N$17: B1.5, IC1.6
- net GND: now also C5.-; no longer C4.-
- net N$15: now also C5.+; no longer C4.+
Routing:
- net GND: track 158.4 -> 275.5 mm
- net N$17: track 0.00 -> 31.5 mm
- net N$15: track 12.2 -> 15.8 mm

Commit message: Add crosshair
Parts:
- moved C2 5.05 mm to (28.6, 39.4)
- moved C5 4.16 mm to (25.2, 34.0)
- moved R1 3.26 mm to (27.4, 44.5)
- moved IC1 2.42 mm to (25.0, 25.0)
- moved R2 1.50 mm to (10.2, 22.9)
- moved LED1 1.50 mm to (35.0, 42.0)
- moved U$1 1.50 mm to (46.4, 35.6)
- moved X2 1.50 mm to (18.5, 7.68)
- moved JP2 1.50 mm to (5.15, 5.14)
- moved JP5 1.50 mm to (10.2, 8.95)
- moved B1 1.50 mm to (10.9, 31.8)
- moved SJ1 1.50 mm to (23.6, 17.8)
- moved X1 1.50 mm to (36.3, 7.68)
- moved C1 1.50 mm to (41.3, 44.5)
- moved JP1 0.99 mm to (40.1, 34.3), flipped to the bottom
Connections:
- net GND: now also IC1.10
Routing:
- net GND: track 275.5 -> 56.7 mm
- net N$14: track 32.3 -> 65.2 mm
- net N$5: track 37.5 -> 62.2 mm, vias 0 -> 1
- net +5V: track 127.7 -> 107.9 mm
- net +12V: track 76.1 -> 62.3 mm
- net N$6: track 30.0 -> 40.4 mm
- net N$8: track 25.2 -> 18.9 mm
- net N$17: track 31.5 -> 35.8 mm
- net N$15: track 15.8 -> 12.2 mm
- net N$9: track 20.7 -> 24.2 mm
- net N$12: track 7.67 -> 4.86 mm
- net N$16: track 7.67 -> 4.86 mm
- net N$13: track 7.67 -> 4.86 mm
- net EN: track 10.4 -> 13.0 mm
- net FEED_HOLD: track 14.6 -> 12.4 mm
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Other:
- board size 50.1 x 48.6 mm -> 49.8 x 49.8 mm

Commit message: Add quadrature encoding X1, X2 and X3 modes
Connections:
- removed net N$5: B1.7, IC1.3
- net N$17: now also IC1.3; no longer IC1.6
- net N$6: now also B1.6; no longer B1.8
Routing:
- net N$5: track 62.2 -> 0.00 mm, vias 1 -> 0
- net N$17: track 35.8 -> 67.3 mm, vias 0 -> 1
- net N$6: track 40.4 -> 45.7 mm
Changed lines of the file:
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@@
 <?xml version="1.0" encoding="utf-8"?>
 <!DOCTYPE eagle SYSTEM "eagle.dtd">
-<eagle version="9.4.0">
+<eagle version="9.4.2">
 <drawing>
 <settings>
@@
 <wire x1="34.925" y1="43.815" x2="34.996421875" y2="43.236065625" width="0.1524" layer="1"/>
 </signal>
-<signal name="N$5">
-<contactref element="IC1" pad="3"/>
-<contactref element="B1" pad="7"/>
-<wire x1="26.035" y1="19.05" x2="26.035" y2="20.955" width="0.1524" layer="16"/>
-<wire x1="22.86" y1="15.875" x2="26.035" y2="19.05" width="0.1524" layer="16"/>
-<wire x1="17.78" y1="10.795" x2="22.86" y2="15.875" width="0.1524" layer="1"/>
-<wire x1="15.875" y1="10.795" x2="17.78" y2="10.795" width="0.1524" layer="1"/>
-<wire x1="12.7" y1="7.62" x2="15.875" y2="10.795" width="0.1524" layer="1"/>
-<wire x1="12.7" y1="3.175" x2="12.7" y2="7.62" width="0.1524" layer="1"/>
-<wire x1="12.065" y1="2.54" x2="12.7" y2="3.175" width="0.1524" layer="1"/>
-<wire x1="3.175" y1="2.54" x2="12.065" y2="2.54" width="0.1524" layer="1"/>
-<wire x1="1.905" y1="3.81" x2="3.175" y2="2.54" width="0.1524" layer="1"/>
-<wire x1="1.905" y1="27.94" x2="1.905" y2="3.81" width="0.1524" layer="1"/>
-<wire x1="3.175" y1="29.21" x2="1.905" y2="27.94" width="0.1524" layer="1"/>
-<wire x1="26.035" y1="20.955" x2="25.93911875" y2="21.15711875" width="0.1524" layer="16"/>
-<wire x1="3.175" y1="29.21" x2="3.246421875" y2="29.266065625" width="0.1524" layer="1"/>
-<via x="22.86" y="15.875" extent="1-16" drill="0.35"/>
-</signal>
 <signal name="N$6">
 <contactref element="IC1" pad="4"/>
-<contactref element="B1" pad="8"/>
 <wire x1="25.4" y1="22.225" x2="25.4" y2="21.59" width="0.1524" layer="16"/>
 <wire x1="26.035" y1="22.86" x2="25.4" y2="22.225" width="0.1524" layer="16"/>
@@
 <wire x1="23.495" y1="13.97" x2="28.575" y2="19.05" width="0.1524" layer="16"/>
 <wire x1="15.875" y1="13.97" x2="23.495" y2="13.97" width="0.1524" layer="16"/>
-<wire x1="3.175" y1="26.67" x2="15.875" y2="13.97" width="0.1524" layer="16"/>
 <wire x1="25.4" y1="21.59" x2="25.28911875" y2="21.15711875" width="0.1524" layer="16"/>
-<wire x1="3.175" y1="26.67" x2="3.246421875" y2="26.726065625" width="0.1524" layer="16"/>
+<contactref element="B1" pad="6"/>
+<wire x1="3.81" y1="30.48" x2="3.81" y2="31.75" width="0.1524" layer="16"/>
+<wire x1="8.89" y1="25.4" x2="3.81" y2="30.48" width="0.1524" layer="16"/>
+<wire x1="8.89" y1="20.955" x2="8.89" y2="25.4" width="0.1524" layer="16"/>
+<wire x1="15.875" y1="13.97" x2="8.89" y2="20.955" width="0.1524" layer="16"/>
+<wire x1="3.81" y1="31.75" x2="3.246421875" y2="31.806065625" width="0.1524" layer="16"/>
 </signal>
 <signal name="N$7">
@@
 </signal>
 <signal name="N$17">
-<contactref element="IC1" pad="6"/>
+<contactref element="IC1" pad="3"/>
 <contactref element="B1" pad="5"/>
-<wire x1="24.13" y1="19.685" x2="24.13" y2="20.955" width="0.1524" layer="16"/>
-<wire x1="19.05" y1="14.605" x2="24.13" y2="19.685" width="0.1524" layer="16"/>
-<wire x1="17.78" y1="14.605" x2="19.05" y2="14.605" width="0.1524" layer="16"/>
-<wire x1="5.08" y1="27.305" x2="17.78" y2="14.605" width="0.1524" layer="16"/>
-<wire x1="5.08" y1="32.385" x2="5.08" y2="27.305" width="0.1524" layer="16"/>
-<wire x1="3.175" y1="34.29" x2="5.08" y2="32.385" width="0.1524" layer="16"/>
-<wire x1="24.13" y1="20.955" x2="23.98911875" y2="21.15711875" width="0.1524" layer="16"/>
-<wire x1="3.175" y1="34.29" x2="3.246421875" y2="34.346065625" width="0.1524" layer="16"/>
+<wire x1="26.035" y1="19.05" x2="26.035" y2="20.955" width="0.1524" layer="16"/>
+<wire x1="22.86" y1="15.875" x2="26.035" y2="19.05" width="0.1524" layer="16"/>
+<wire x1="17.78" y1="10.795" x2="22.86" y2="15.875" width="0.1524" layer="1"/>
+<wire x1="15.875" y1="10.795" x2="17.78" y2="10.795" width="0.1524" layer="1"/>
+<wire x1="12.7" y1="7.62" x2="15.875" y2="10.795" width="0.1524" layer="1"/>
+<wire x1="12.7" y1="3.175" x2="12.7" y2="7.62" width="0.1524" layer="1"/>
+<wire x1="12.065" y1="2.54" x2="12.7" y2="3.175" width="0.1524" layer="1"/>
+<wire x1="3.175" y1="2.54" x2="12.065" y2="2.54" width="0.1524" layer="1"/>
+<wire x1="1.905" y1="3.81" x2="3.175" y2="2.54" width="0.1524" layer="1"/>
+<wire x1="1.905" y1="33.02" x2="1.905" y2="3.81" width="0.1524" layer="1"/>
+<wire x1="26.035" y1="20.955" x2="25.93911875" y2="21.15711875" width="0.1524" layer="16"/>
+<via x="22.86" y="15.875" extent="1-16" drill="0.35"/>
+<wire x1="1.905" y1="33.02" x2="3.175" y2="34.29" width="0.1524" layer="1"/>
+<wire x1="3.175" y1="34.29" x2="3.246421875" y2="34.346065625" width="0.1524" layer="1"/>
 </signal>
 </signals>
